File: STM32F042F6P6_Breakout.kicad_pcb (KiCad board)
At the start: 2 copper layers, 20.3 x 25.4 mm, 24 parts, among them J1 Conn_01x10_Male, J2 USB_B_Micro, J3 Conn_01x10_Male, J4 Conn_01x04_Male, Q1 Q_NPN, SW1 SW_Push, U1 TLV70033_SOT23-5, U2 STM32F042F6Px

Commit message: rev 1.1
Parts:
- SW1: footprint Button_Switch_SMD:SW_SPST_FSMSM -> Local:SW_SPST_FSMSM
- moved SW1 0.10 mm to (150.0, 93.4)
Routing:
- net GND: track 84.9 -> 116.5 mm, vias 13 -> 19
- net SWCLK: track 30.5 -> 31.6 mm
- net /VBUS: track 21.4 -> 22.3 mm
